Commit message: update sail lower/upper limit

File: usv_sim/xacro/sailboat.xacro (robot description, xacro)
@@ -40,5 +40,5 @@
         <dynamics damping="1.0"/>
         <axis xyz="0 0 1"/>
-        <limit effort="100" velocity="70" lower="-${PI}" upper="${PI}" />
+        <limit effort="100" velocity="70" lower="${-PI/2}" upper="${PI/2}" />
     </joint>
     <link name="keel">

Commit message: fix: joint limit

File: usv_sim/xacro/sailboat.xacro (robot description, xacro)
@@ -40,5 +40,5 @@
         <dynamics damping="1.0"/>
         <axis xyz="0 0 1"/>
-        <limit effort="100" velocity="70" lower="${-PI/2}" upper="${PI/2}" />
+        <limit effort="100" velocity="70" lower="-${PI}" upper="${PI}" />
     </joint>
     <link name="keel">

Commit message: fix: change sailboat configuration to avoid oscillations

File: usv_sim/xacro/sailboat.xacro (robot description, xacro)
@@ -40,5 +40,5 @@
         <dynamics damping="1.0"/>
         <axis xyz="0 0 1"/>
-        <limit effort="100" velocity="70" lower="-${PI}" upper="${PI}" />
+        <limit effort="1000" velocity="70" lower="-${PI/2}" upper="${PI/2}" />
     </joint>
     <link name="keel">

Commit message: fix: change sailboat configuration to avoid oscillations [1]

File: usv_sim/xacro/sailboat.xacro (robot description, xacro)
@@ -40,5 +40,5 @@
         <dynamics damping="1.0"/>
         <axis xyz="0 0 1"/>
-        <limit effort="1000" velocity="70" lower="-${PI/2}" upper="${PI/2}" />
+        <limit effort="500" velocity="${PI}" lower="-${PI/2}" upper="${PI/2}" />
     </joint>
     <link name="keel">

Commit message: Added a framework to easily tweak the simulation for the gym environment and improved sail performance at higher wind speeds

File: usv_sim/xacro/sailboat.xacro (robot description, xacro)
@@ -14,10 +14,10 @@
 			<mass value="1" />
 			<inertia
-			  ixx="0.4708"
+			  ixx="47080"
 			  ixy="0.0"
-			  iyy="0.5208"
+			  iyy="52080"
 			  ixz="0.0"
 			  iyz="0.0"
-			  izz="0.0508"/>
+			  izz="5000.8"/>
 		</inertial>
 	    <collision name="collision">
@@ -40,5 +40,5 @@
         <dynamics damping="1.0"/>
         <axis xyz="0 0 1"/>
-        <limit effort="500" velocity="${PI}" lower="-${PI/2}" upper="${PI/2}" />
+        <limit effort="1000000" velocity="2" lower="-${PI/2}" upper="${PI/2}" />
     </joint>
     <link name="keel">
@@ -72,5 +72,5 @@
         <dynamics damping="1.0"/>
         <axis xyz="0 0 1"/>
-        <limit effort="30" velocity="5" lower="0" upper="0" />
+        <limit effort="300" velocity="5" lower="0" upper="0" />
     </joint>
     <!-- Plugin list -->

Commit message: Fixed Dockerfile to actually build everything, fixed sim parameters to go super fast, and added cleanup to the build_sim.sh script

File: usv_sim/xacro/sailboat.xacro (robot description, xacro)
@@ -14,10 +14,10 @@
 			<mass value="1" />
 			<inertia
-			  ixx="47080"
+			  ixx="470.80"
 			  ixy="0.0"
-			  iyy="52080"
+			  iyy="520.80"
 			  ixz="0.0"
 			  iyz="0.0"
-			  izz="5000.8"/>
+			  izz="500"/>
 		</inertial>
 	    <collision name="collision">
@@ -40,5 +40,5 @@
         <dynamics damping="1.0"/>
         <axis xyz="0 0 1"/>
-        <limit effort="1000000" velocity="2" lower="-${PI/2}" upper="${PI/2}" />
+        <limit effort="1000" velocity="2" lower="-${PI/2}" upper="${PI/2}" />
     </joint>
     <link name="keel">

Commit message: Removed README.md

File: usv_sim/xacro/sailboat.xacro (robot description, xacro)
@@ -14,10 +14,10 @@
 			<mass value="1" />
 			<inertia
-			  ixx="470.80"
+			  ixx="0.4708"
 			  ixy="0.0"
-			  iyy="520.80"
+			  iyy="0.5208"
 			  ixz="0.0"
 			  iyz="0.0"
-			  izz="500"/>
+			  izz="0.0508"/>
 		</inertial>
 	    <collision name="collision">
@@ -40,5 +40,5 @@
         <dynamics damping="1.0"/>
         <axis xyz="0 0 1"/>
-        <limit effort="1000" velocity="2" lower="-${PI/2}" upper="${PI/2}" />
+        <limit effort="100000" velocity="1" lower="-${PI/2}" upper="${PI/2}" />
     </joint>
     <link name="keel">
@@ -72,5 +72,5 @@
         <dynamics damping="1.0"/>
         <axis xyz="0 0 1"/>
-        <limit effort="300" velocity="5" lower="0" upper="0" />
+        <limit effort="30" velocity="5" lower="0" upper="0" />
     </joint>
     <!-- Plugin list -->
